Commit message: change param for yawrate

File: amr_description/ardrone.xacro (robot description, xacro)
@@ -1,17 +1,14 @@
 <?xml version="1.0"?>
-<robot name="iris" xmlns:xacro="http://ros.org/wiki/xacro">
+<robot name="ardrone" xmlns:xacro="http://ros.org/wiki/xacro">
   <!-- Properties -->
-  <xacro:property name="namespace" value="iris" />
+  <xacro:property name="namespace" value="ardrone" />
   <xacro:property name="rotor_velocity_slowdown_sim" value="10" />
   <xacro:property name="use_mesh_file" value="true" />
-  <xacro:property name="mesh_file" value="package://rotors_description/meshes/iris.dae" />
+  <xacro:property name="mesh_file" value="package://rotors_description/meshes/ardrone.dae" />
   <xacro:property name="mass" value="1.5" /> <!-- [kg] -->
-  <xacro:property name="body_width" value="0.47" /> <!-- [m] -->
-  <xacro:property name="body_height" value="0.11" /> <!-- [m] -->
+  <xacro:property name="body_width" value="0.3" /> <!-- [m] -->
+  <xacro:property name="body_height" value="0.16" /> <!-- [m] -->
   <xacro:property name="mass_rotor" value="0.005" /> <!-- [kg] -->
-  <xacro:property name="arm_length_front_x" value="0.13" /> <!-- [m] -->
-  <xacro:property name="arm_length_back_x" value="0.13" /> <!-- [m] -->
-  <xacro:property name="arm_length_front_y" value="0.22" /> <!-- [m] -->
-  <xacro:property name="arm_length_back_y" value="0.2" /> <!-- [m] -->
+  <xacro:property name="arm_length" value="0.09" /> <!-- [m] -->
   <xacro:property name="rotor_offset_top" value="0.023" /> <!-- [m] -->
   <xacro:property name="radius_rotor" value="0.1" /> <!-- [m] -->
@@ -35,8 +32,8 @@
   </xacro:property>
   <!-- Included URDF Files -->
-  <xacro:include filename="$(find amr_description)/multirotor_base.xacro" />
+  <xacro:include filename="$(find rotors_description)/urdf/multirotor_base.xacro" />
   <!-- Instantiate multirotor_base_macro once -->
   <xacro:multirotor_base_macro
-    robot_namespace="iris"
+    robot_namespace="ardrone"
     mass="${mass}"
     body_width="${body_width}"
@@ -49,10 +46,10 @@
   <!-- Instantiate rotors -->
   <xacro:vertical_rotor
-    robot_namespace="iris"
+    robot_namespace="ardrone"
     suffix="front_right"
     direction="ccw"
     motor_constant="${motor_constant}"
     moment_constant="${moment_constant}"
-    parent="iris/base_link"
+    parent="ardrone/base_link"
     mass_rotor="${mass_rotor}"
     radius_rotor="${radius_rotor}"
@@ -63,17 +60,17 @@
     rotor_drag_coefficient="${rotor_drag_coefficient}"
     rolling_moment_coefficient="${rolling_moment_coefficient}"
-    color="Blue"
+    color="Red"
     use_own_mesh="false"
     mesh="">
-    <origin xyz="${arm_length_front_x} -${arm_length_front_y} ${rotor_offset_top}" rpy="0 0 0" />
+    <origin xyz="${sqrt2 * arm_length} -${sqrt2 * arm_length} ${rotor_offset_top}" rpy="0 0 0" />
     <xacro:insert_block name="rotor_inertia" />
   </xacro:vertical_rotor>
   <xacro:vertical_rotor
-    robot_namespace="iris"
+    robot_namespace="ardrone"
     suffix="back_left"
     direction="ccw"
     motor_constant="${motor_constant}"
     moment_constant="${moment_constant}"
-    parent="iris/base_link"
+    parent="ardrone/base_link"
     mass_rotor="${mass_rotor}"
     radius_rotor="${radius_rotor}"
@@ -84,16 +81,16 @@
     rotor_drag_coefficient="${rotor_drag_coefficient}"
     rolling_moment_coefficient="${rolling_moment_coefficient}"
-    color="Red"
+    color="Blue"
     use_own_mesh="false"
     mesh="">
-    <origin xyz="-${arm_length_back_x} ${arm_length_back_y} ${rotor_offset_top}" rpy="0 0 0" />
+    <origin xyz="-${sqrt2 * arm_length} ${sqrt2 * arm_length} ${rotor_offset_top}" rpy="0 0 0" />
     <xacro:insert_block name="rotor_inertia" />
   </xacro:vertical_rotor>
-  <xacro:vertical_rotor robot_namespace="iris"
+  <xacro:vertical_rotor robot_namespace="ardrone"
     suffix="front_left"
     direction="cw"
     motor_constant="${motor_constant}"
     moment_constant="${moment_constant}"
-    parent="iris/base_link"
+    parent="ardrone/base_link"
     mass_rotor="${mass_rotor}"
     radius_rotor="${radius_rotor}"
@@ -104,16 +101,16 @@
     rotor_drag_coefficient="${rotor_drag_coefficient}"
     rolling_moment_coefficient="${rolling_moment_coefficient}"
-    color="Blue"
+    color="Red"
     use_own_mesh="false"
     mesh="">
-    <origin xyz="${arm_length_front_x} ${arm_length_front_y} ${rotor_offset_top}" rpy="0 0 0" />
+    <origin xyz="${sqrt2 * arm_length} ${sqrt2 * arm_length} ${rotor_offset_top}" rpy="0 0 0" />
     <xacro:insert_block name="rotor_inertia" />
   </xacro:vertical_rotor>
-  <xacro:vertical_rotor robot_namespace="iris"
+  <xacro:vertical_rotor robot_namespace="ardrone"
     suffix="back_right"
     direction="cw"
     motor_constant="${motor_constant}"
     moment_constant="${moment_constant}"
-    parent="iris/base_link"
+    parent="ardrone/base_link"
     mass_rotor="${mass_rotor}"
     radius_rotor="${radius_rotor}"
@@ -124,8 +121,8 @@
     rotor_drag_coefficient="${rotor_drag_coefficient}"
     rolling_moment_coefficient="${rolling_moment_coefficient}"
-    color="Red"
+    color="Blue"
     use_own_mesh="false"
     mesh="">
-    <origin xyz="-${arm_length_back_x} -${arm_length_back_y} ${rotor_offset_top}" rpy="0 0 0" />
+    <origin xyz="-${sqrt2 * arm_length} -${sqrt2 * arm_length} ${rotor_offset_top}" rpy="0 0 0" />
     <xacro:insert_block name="rotor_inertia" />
   </xacro:vertical_rotor>

File: amr_description/ardrone_base.xacro (robot description, xacro)
@@ -1,16 +1,16 @@
 <?xml version="1.0"?>
-<robot name="iris" xmlns:xacro="http://ros.org/wiki/xacro">
-  <xacro:include filename="$(find amr_description)/component_snippets.xacro" />
-  <!-- Instantiate iris "mechanics" -->
-  <xacro:include filename="$(find amr_description)/iris.xacro" />
+<robot name="ardrone" xmlns:xacro="http://ros.org/wiki/xacro">
+  <xacro:include filename="$(find rotors_description)/urdf/component_snippets.xacro" />
+  <!-- Instantiate ardrone "mechanics" -->
+  <xacro:include filename="$(find rotors_description)/urdf/ardrone.xacro" />
   <!-- Instantiate a controller. -->
-  <xacro:controller_plugin_macro namespace="iris" imu_sub_topic="imu" />
+  <xacro:controller_plugin_macro namespace="ardrone" imu_sub_topic="imu" />
   <xacro:if value="$(arg enable_mavlink_interface)">
     <!-- Instantiate mavlink telemetry interface. -->
-    <xacro:default_mavlink_interface namespace="iris" imu_sub_topic="imu" rotor_count="4" />
+    <xacro:default_mavlink_interface namespace="ardrone" imu_sub_topic="imu" rotor_count="4" />
   </xacro:if>
   <xacro:camera_macro
-    namespace="iris"
-    parent_link="iris/base_link"
+    namespace="ardrone"
+    parent_link="ardrone/base_link"
     camera_suffix="front"
     frame_rate="30.0"
@@ -26,9 +26,9 @@
     >
     <box size="0.02 0.02 0.02" />
-    <origin xyz="0.10 0 0" rpy="0 0 0"/>
+    <origin xyz="0.06 0 0" rpy="0 0 0"/>
   </xacro:camera_macro>
   <xacro:camera_macro
-    namespace="iris"
-    parent_link="iris/base_link"
+    namespace="ardrone"
+    parent_link="ardrone/base_link"
     camera_suffix="bottom"
     frame_rate="30.0"
@@ -47,12 +47,12 @@
   </xacro:camera_macro>
   <!-- Mount an ADIS16448 IMU. -->
-  <xacro:default_imu namespace="iris" parent_link="iris/base_link" />
+  <xacro:default_imu namespace="ardrone" parent_link="ardrone/base_link" />
   <xacro:if value="$(arg enable_ground_truth)">
-    <xacro:ground_truth_imu_and_odometry namespace="iris" parent_link="iris/base_link" />
+    <xacro:ground_truth_imu_and_odometry namespace="ardrone" parent_link="ardrone/base_link" />
   </xacro:if>
   <xacro:if value="$(arg enable_logging)">
     <!-- Instantiate a logger -->
     <xacro:bag_plugin_macro
-      namespace="iris"
+      namespace="ardrone"
       bag_file="$(arg log_file)"
       rotor_velocity_slowdown_sim="${rotor_velocity_slowdown_sim}"
